File: chuniAir/chuniAir.kicad_pcb (KiCad board)
At the start: 2 copper layers, 50.8 x 51.3 mm, 11 parts, among them U1 ProMicro

Commit message: update
Parts:
- removed REF** (x3): MountingHole_3.2mm_M3, MountingHole:MountingHole_3.2mm_M3
- removed U1: ProMicro, promicro:ProMicro-EnforcedTop
- added H1: MountingHole, MountingHole:MountingHole_4.3mm_M4, F.Cu at (165.6, 36.1)
- added H2: MountingHole, MountingHole:MountingHole_4.3mm_M4, F.Cu at (205.5, 36.0)
- added H3: MountingHole, MountingHole:MountingHole_4.3mm_M4, F.Cu at (165.6, 98.0)
- added H4: MountingHole, MountingHole:MountingHole_4.3mm_M4, F.Cu at (205.5, 98.0)
- added U2: Elite-C, PCM_marbastlib-xp-promicroish:Elite-C_ACH, F.Cu at (185.3, 60.5)
- moved Power1 92.0 mm to (184.3, 92.0)
- moved Left_Sensor1 89.8 mm to (168.2, 58.4)
- moved Left_LED1 89.8 mm to (168.2, 89.1)
- moved Left_Sensor2 89.8 mm to (168.2, 77.3)
- moved Right_LED1 84.9 mm to (202.1, 84.1)
- moved Right_Sensor1 84.9 mm to (202.1, 45.9)
- moved Right_Sensor2 84.9 mm to (202.1, 64.8)
Routing:
- net +12V: track 96.1 -> 42.2 mm
- net /DATA1: track 31.8 -> 75.4 mm
- net /TWR4: track 42.8 -> 34.3 mm
- net /TWR5: track 42.4 -> 34.3 mm
- net /OUT4: track 32.8 -> 25.3 mm
- net /OUT6: track 32.9 -> 25.3 mm
- net /OUT5: track 32.8 -> 25.3 mm
- net /DATA2: track 32.2 -> 39.7 mm
- net /TWR6: track 41.1 -> 34.6 mm
- net /TWR3: track 40.2 -> 34.3 mm
- net /TWR2: track 40.2 -> 34.4 mm
- net /TWR1: track 39.9 -> 34.4 mm
- net /OUT1: track 9.13 -> 12.4 mm
- net /OUT2: track 9.07 -> 12.3 mm
- net /OUT3: track 9.50 -> 12.2 mm
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Other:
- board size 50.8 x 51.3 mm -> 49 x 71 mm
- board text added: "air string rev1.0"
