File: chuniAir/chuniAir.kicad_sch (KiCad schematic)
At the start: 8 parts, among them U1 ProMicro

Commit message: update
Parts:
- removed U1: ProMicro, promicro:ProMicro-EnforcedTop, symbol promicro:ProMicro
- added H1, H2, H3, H4: MountingHole, MountingHole:MountingHole_4.3mm_M4, symbol Mechanical:MountingHole
- added U2: Elite-C, PCM_marbastlib-xp-promicroish:Elite-C_ACH, symbol PCM_marbastlib-promicroish:Elite-C
Connections:
- net +5V: now also U2.16 (VCC)
- net DATA1: now also U2.19 (F6)
- net DATA2: now also U2.20 (F7)
- net GND: now also U2.3 (GND), U2.4 (GND)
- net OUT1: now also U2.7 (D4)
- net OUT2: now also U2.8 (C6)
- net OUT3: now also U2.9 (D7)
- net OUT4: now also U2.10 (E6)
- net OUT5: now also U2.11 (B4)
- net OUT6: now also U2.12 (B5)
